Commit message: Updated the xacro file so the wheels turned regularly and updated launch file

File: urdf/robot_links_and_joints.xacro (robot description, xacro)
@@ -47,4 +47,5 @@
 		</link>
 		<joint name="base_wheel_${suffix}_joint" type="continuous">
+			<axis xyz="0 0 1" />
 			<parent link="base"/>
 			<child link="wheel_${suffix}"/>
@@ -69,4 +70,5 @@
 		</link>
 		<joint name="base_wheel_${suffix}_joint" type="continuous">
+			<axis xyz="0 0 1" />
 			<parent link="base"/>
 			<child link="wheel_${suffix}"/>

File: urdf/urdf_from_xacro.urdf (robot description, URDF)
Before this commit: robot anh_robot, 8 links, 11 joints
Joints:
- joint base_wheel_center_joint: axis (none) -> 0 0 1
- joint base_wheel_left_joint: axis (none) -> 0 0 1
- joint base_wheel_right_joint: axis (none) -> 0 0 1
